File: Mini_GPS_IMU/MiniGPSIMU.sch (KiCad schematic (older format))
At the start: 26 parts, among them J1 CONN_01X04_MALE, SW1 SW_Push, U1 TCR2LE33LM, U2 STM32F072CBUx

Commit message: Finished version 1.0 of GPS Diamond.
Parts:
- removed C1, C2: 0.1uF, Capacitors_SMD:C_0402_NoSilk, symbol C
- removed R2: 10k, Resistors_SMD:R_0402_NoSilk, symbol R
- removed U2: STM32F072CBUx, Housings_DFN_QFN:QFN-48-1EP_7x7mm_Pitch0.5mm, symbol STM32F072CBUx
- added B2: SW_Push, Buttons_Switches_SMD:SW_SPST_B3U-3000P, symbol SW_Push
- added C14: 100nF, Capacitors_SMD:C_0402, symbol C
- added R6, R8: 10K, Resistors_SMD:R_0402, symbol R
- added U2: STM32F042K6Ux, local:UFQFPN32, symbol STM32F042K6Ux
- B1: renamed from SW1; footprint Buttons_Switches_SMD:SW_SPST_B3U-1000P -> jumper:SOLDER-JUMPER_1-WAY
- C3: value 4.7uF -> 1uF; footprint Capacitors_SMD:C_0402_NoSilk -> Capacitors_SMD:C_0402
- C4: value 100nF -> 10nF; footprint Capacitors_SMD:C_0402_NoSilk -> Capacitors_SMD:C_0402
- C5, C6, C7: footprint Capacitors_SMD:C_0402_NoSilk -> Capacitors_SMD:C_0402
- C8: value 10nF -> 100nF; footprint Capacitors_SMD:C_0402_NoSilk -> Capacitors_SMD:C_0402
- C9: value 1uF -> 4.7uF; footprint Capacitors_SMD:C_0402_NoSilk -> Capacitors_SMD:C_0402
- R1, R3, R4, R7: footprint Resistors_SMD:R_0402_NoSilk -> Resistors_SMD:R_0402
- renumbered NRST1 to J2, GND1 to J3, SWDIO1 to J5, SWDCLK1 to J6
Connections:
- net +3V3: now also B2.2, C14.1, R6.2, R8.2, U2.1 (VDD), U2.17 (VDDIO2), U2.5 (VDDA); no longer C5.1
- net +5V: now also C5.1
- net GND: now also U1.2 (GND), C14.2, U2.33 (VSS)
- net LED: now also U2.11 (ADC_IN5/CEC/I2S1_CK/SPI1_SCK/TIM2_CH1/TIM2_ETR/TSC_G2_IO2/PA5)
- net at J5.1: now also U2.23 (IR_OUT/SYS_SWDIO/USB_OE/PA13)
- net at J6.1: now also U2.24 (SYS_SWCLK/USART2_TX/PA14)
- net at B1.2, R7.1: now also U2.31 (PF11)
- net at J2.1: now also U2.4 (NRST)
- net UART1_RX renamed USART1_RX
- net USART1_RX: now also U2.20 (I2C1_SDA/TIM17_BKIN/TIM1_CH3/TSC_G4_IO2/USART1_RX/PA10)
- net UART1_TX renamed USART1_TX
- net USART1_TX: now also U2.19 (I2C1_SCL/TIM1_CH2/TSC_G4_IO1/USART1_TX/PA9)
- new net: B2.1, U2.10 (ADC_IN4/I2S1_WS/SPI1_NSS/TIM14_CH1/TSC_G2_IO1/USART2_CK/USB_OE/PA4)
- new net I2C1_SCL: R6.1, U2.29 (PB6/I2C1_SCL/TIM16_CH1N/TSC_G5_IO3/USART1_TX)
- new net I2C1_SDA: R8.1, U2.30 (PB7/I2C1_SDA/TIM17_CH1N/TSC_G5_IO4/USART1_RX)
- new net IMU_INT1: U2.6 (ADC_IN0/RTC_TAMP2/SYS_WKUP1/TIM2_CH1/TIM2_ETR/TSC_G1_IO1/USART2_CTS/PA0)
- new net IMU_INT2: U2.7 (ADC_IN1/TIM2_CH2/TSC_G1_IO2/USART2_DE/USART2_RTS/PA1)
- new net USART2_RX: U2.9 (ADC_IN3/TIM2_CH4/TSC_G1_IO4/USART2_RX/PA3)
- new net USART2_TX: U2.8 (ADC_IN2/SYS_WKUP4/TIM2_CH3/TSC_G1_IO3/USART2_TX/PA2)
- no-connect marks 22 -> 15
Other:
- moved on the sheet: B1, C3, C4, C6, C7, C8, C9, D2, J2, J5, J6, R1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
