File: Dual_Inverter/Dual_Inverter.sch (KiCad schematic (older format))
At the start: 10 parts, among them J1 CONN_01X04_MALE, J2 CONN_01X04_MALE, U1 MCP1754ST-3302E/MB-SOT-23, U2 NC7WZ14P6X

Commit message: Fixes a trace connection on the Dual Inverter and makes the solder jumper pads smaller.
Parts:
- A1, A2, B1, B2: footprint jumper:SOLDER-JUMPER_2-WAY -> local:SOLDER-JUMPER_2-WAY
Changed lines of the file:
@@
 F 0 "A1" H 3350 4750 60  0000 C CNN
 F 1 "JUMPER_3-PIN" V 3050 4650 60  0000 C CNN
-F 2 "jumper:SOLDER-JUMPER_2-WAY" H 3200 4650 60  0001 C CNN
+F 2 "local:SOLDER-JUMPER_2-WAY" H 3200 4650 60  0001 C CNN
 F 3 "" H 3350 4750 60  0001 C CNN
 	1    3350 4650
@@
 F 0 "B1" H 3350 5300 60  0000 C CNN
 F 1 "JUMPER_3-PIN" V 3650 5200 60  0000 C CNN
-F 2 "jumper:SOLDER-JUMPER_2-WAY" H 3200 5200 60  0001 C CNN
+F 2 "local:SOLDER-JUMPER_2-WAY" H 3200 5200 60  0001 C CNN
 F 3 "" H 3350 5300 60  0001 C CNN
 	1    3350 5200
@@
 F 0 "B2" H 5400 5300 60  0000 C CNN
 F 1 "JUMPER_3-PIN" V 5100 5200 60  0000 C CNN
-F 2 "jumper:SOLDER-JUMPER_2-WAY" H 5250 5200 60  0001 C CNN
+F 2 "local:SOLDER-JUMPER_2-WAY" H 5250 5200 60  0001 C CNN
 F 3 "" H 5400 5300 60  0001 C CNN
 	1    5400 5200
@@
 F 0 "A2" H 5400 4750 60  0000 C CNN
 F 1 "JUMPER_3-PIN" V 5700 4650 60  0000 C CNN
-F 2 "jumper:SOLDER-JUMPER_2-WAY" H 5250 4650 60  0001 C CNN
+F 2 "local:SOLDER-JUMPER_2-WAY" H 5250 4650 60  0001 C CNN
 F 3 "" H 5400 4750 60  0001 C CNN
 	1    5400 4650
