File: LPLink_Nano/LPLink_Nano.kicad_pcb (KiCad board)
At the start: 2 copper layers, 25 x 17 mm, 36 parts, among them J1 USB_OTG, J2 CONN_COAXIAL, J3 CONN_01X04_MALE, J4 CONN_01X04_MALE, J5 CONN_01X01_MALE, J6 CONN_01X01_MALE, J7 CONN_01X01_MALE, J8 CONN_01X01_MALE, SW1 SW_Push, U1 RFM22, U2 STM32F303CC, U3 MIC5353-3.3YMT-TR, Y1 Ceralock

Commit message: LPLink Nano V1.0.
Parts:
- moved R3 4.17 mm to (160.6, 101.2), turned to 180 degrees
- moved R5 2.16 mm to (160.6, 99.2), turned to 180 degrees
- moved R4 1.21 mm to (160.6, 100.2), turned to 180 degrees
- moved D3 0.30 mm to (160.8, 104.4)
- moved D2 0.25 mm to (160.8, 105.8)
- moved D4 0.25 mm to (160.8, 103.0)
- moved D5 0.25 mm to (160.8, 107.2)
- moved J3 0.05 mm to (159.6, 103.9)
- moved J4 0.05 mm to (159.6, 95.9)
Routing:
- net GND: track 27.5 -> 36.0 mm, vias 16 -> 15
- net Net-(J3-Pad4): track 16.3 -> 10.3 mm
- net Net-(D2-Pad2): track 1.64 -> 6.09 mm
- net Net-(D4-Pad2): track 1.77 -> 5.38 mm
- net Net-(R3-Pad2): track 8.12 -> 5.17 mm
- net Net-(D3-Pad2): track 4.19 -> 6.02 mm
- net Net-(R5-Pad2): track 6.56 -> 4.95 mm
Other:
- board text added: "+5"
- board text added: "Boot"
- board text added: "Flexi"
- board text added: "GND"
- board text added: "LPLink Nano V1.0"
- board text added: "Link"
- board text added: "Main"
- board text added: "Pwr"
- board text added: "Rx"
- board text added: "Tx"

Commit message: Adds a BOM o LPLink Nano.
Parts:
- C10, C8, C9: value 100nF -> 0.1uF
- D2: value LED -> Blue
- D3: value LED -> Red
- D4: value LED -> Yellow
- D5: value LED -> Green
- R1, R2: value 2.2k -> 22R
- R3, R4, R5, R6: value R -> 100R
Changed lines of the file:
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@@
       (effects (font (size 0.5 0.5) (thickness 0.1)) (justify mirror))
     )
-    (fp_text value LED (at 0 -1.4 180) (layer B.Fab)
+    (fp_text value Blue (at 0 -1.4 180) (layer B.Fab)
       (effects (font (size 1 1) (thickness 0.15)) (justify mirror))
     )
@@
       (effects (font (size 0.5 0.5) (thickness 0.1)) (justify mirror))
     )
-    (fp_text value LED (at 0 -1.4 180) (layer B.Fab)
+    (fp_text value Red (at 0 -1.4 180) (layer B.Fab)
       (effects (font (size 1 1) (thickness 0.15)) (justify mirror))
     )
@@
       (effects (font (size 0.5 0.5) (thickness 0.1)) (justify mirror))
     )
-    (fp_text value LED (at 0 -1.4 180) (layer B.Fab)
+    (fp_text value Yellow (at 0 -1.4 180) (layer B.Fab)
       (effects (font (size 1 1) (thickness 0.15)) (justify mirror))
     )
@@
       (effects (font (size 0.5 0.5) (thickness 0.1)) (justify mirror))
     )
-    (fp_text value LED (at 0 -1.4 180) (layer B.Fab)
+    (fp_text value Green (at 0 -1.4 180) (layer B.Fab)
       (effects (font (size 1 1) (thickness 0.15)) (justify mirror))
     )
@@
       (effects (font (size 0.5 0.5) (thickness 0.1)))
     )
-    (fp_text value 2.2k (at 0 1.45) (layer F.Fab)
+    (fp_text value 22R (at 0 1.45) (layer F.Fab)
       (effects (font (size 1 1) (thickness 0.15)))
     )
@@
       (effects (font (size 0.5 0.5) (thickness 0.1)))
     )
-    (fp_text value 2.2k (at 0 1.45) (layer F.Fab)
+    (fp_text value 22R (at 0 1.45) (layer F.Fab)
       (effects (font (size 1 1) (thickness 0.15)))
     )
@@
       (effects (font (size 0.5 0.5) (thickness 0.1)) (justify mirror))
     )
-    (fp_text value R (at 0 -1.45 180) (layer B.Fab)
+    (fp_text value 100R (at 0 -1.45 180) (layer B.Fab)
       (effects (font (size 1 1) (thickness 0.15)) (justify mirror))
     )
@@
       (effects (font (size 0.5 0.5) (thickness 0.1)) (justify mirror))
     )
-    (fp_text value R (at 0 -1.45 180) (layer B.Fab)
+    (fp_text value 100R (at 0 -1.45 180) (layer B.Fab)
       (effects (font (size 1 1) (thickness 0.15)) (justify mirror))
     )
@@
       (effects (font (size 0.5 0.5) (thickness 0.1)) (justify mirror))
     )
-    (fp_text value R (at 0 -1.45 180) (layer B.Fab)
+    (fp_text value 100R (at 0 -1.45 180) (layer B.Fab)
       (effects (font (size 1 1) (thickness 0.15)) (justify mirror))
     )
@@
       (effects (font (size 0.5 0.5) (thickness 0.1)) (justify mirror))
     )
-    (fp_text value R (at 0 -1.45 90) (layer B.Fab)
+    (fp_text value 100R (at 0 -1.45 90) (layer B.Fab)
       (effects (font (size 1 1) (thickness 0.15)) (justify mirror))
     )
@@
       (effects (font (size 0.5 0.5) (thickness 0.1)))
     )
-    (fp_text value 100nF (at 0 1.27 270) (layer F.Fab)
+    (fp_text value 0.1uF (at 0 1.27 270) (layer F.Fab)
       (effects (font (size 1 1) (thickness 0.15)))
     )
@@
       (effects (font (size 0.5 0.5) (thickness 0.1)))
     )
-    (fp_text value 100nF (at 0 1.27) (layer F.Fab)
+    (fp_text value 0.1uF (at 0 1.27) (layer F.Fab)
       (effects (font (size 1 1) (thickness 0.15)))
     )
@@
       (effects (font (size 0.5 0.5) (thickness 0.1)))
     )
-    (fp_text value 100nF (at 0 1.27 90) (layer F.Fab)
-      (effects (font (size 1 1) (thickness 0.15)))
-    )
+    (fp_text value 0.1uF (at 0 1.27 90) (layer F.Fab)
+      (effects (font (size 1 1) (thickness 0.15)))
+    )
